File: hardware/KiCAD/meross.kicad_pcb (KiCad board)
At the start: 4 copper layers, 81.5 x 55 mm, 43 parts, among them J1 Conn_01x01_Female, J2 Conn_01x01_Female, J3 Conn_01x04_Male, J4 Conn_01x01_Female, J5 Conn_01x01_Female, J6 Conn_01x01_Female, J7 Conn_01x01_Female, K1 G5Q-1A, K2 G5Q-1A, K3 G5Q-1A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

Commit message: v1.0.0
Parts:
- removed C7: 220uf, Capacitor_THT:CP_Radial_D6.3mm_P2.50mm
- removed D1: D_0001, DVB_LED:LED_0603-red
- removed L1: L_0004, DVB_Inductors:L_2020-Vishay
- removed R6: R_0027, DVB_Resistors:R_0603
- C1, C3, R1, R4: moved to B.Cu
- J3: footprint Connector_PinHeader_2.54mm:PinHeader_1x04_P2.54mm_Vertical -> Connector_PinHeader_2.54mm:PinHeader_2x02_P2.54mm_Vertical
- moved R5 31.0 mm to (124.5, 78.3), turned to 180 degrees
- moved J3 30.8 mm to (131.2, 75.6), turned to 90 degrees
- moved R1 28.1 mm to (141.0, 105.5), turned to 180 degrees
- moved SW1 27.9 mm to (141.0, 104.5), turned to 180 degrees
- moved SW2 26.6 mm to (141.0, 99.5), turned to 180 degrees
- moved C1 26.3 mm to (141.0, 103.5), turned to 180 degrees
- moved C3 26.0 mm to (141.0, 100.5), turned to 180 degrees
- moved R4 12.5 mm to (141.0, 98.4), turned to 180 degrees
- moved U2 12.3 mm to (150.1, 99.2)
- moved C2 12.3 mm to (153.1, 98.9)
- moved C5 12.3 mm to (147.1, 99.4)
- moved C6 12.3 mm to (150.3, 102.2)
- moved R7 9.62 mm to (160.5, 79.0), turned to 0 degrees
- moved Q1 9.30 mm to (160.5, 76.0), turned to 90 degrees
- moved R8 9.18 mm to (160.5, 90.5), turned to 0 degrees
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Connections:
- J3 pad 2: /Rx -> +3.3V
- J3 pad 4: +3.3V -> /Rx
- PS1 pad 5: Net-(L1-Pad1) -> +12V
- R4 pad 2: /Tx -> /GPIO0
- R5 pad 2: /Rx -> Net-(R5-Pad2)
- SW1 pad 1: (no net) -> /RST
- SW1 pad 4: (no net) -> GND
- SW2 pad 1: (no net) -> /GPIO0
- SW2 pad 4: (no net) -> GND
- U1 pad 17: (no net) -> Net-(R5-Pad2)
- U1 pad 20: Net-(D1-Pad1) -> (no net)
Routing:
- net /L: track 39.0 -> 80.2 mm
- net +12V: track 36.5 -> 76.8 mm
- net Net-(D1-Pad1): track 17.1 -> 0.00 mm, vias 2 -> 0
- net /G1: track 46.3 -> 30.1 mm
- net /GPIO0: track 19.3 -> 34.4 mm
- net Net-(R5-Pad2): track 0.00 -> 13.0 mm, vias 0 -> 2
- net Net-(L1-Pad1): track 9.34 -> 0.00 mm
- net /N: track 0.00 -> 8.43 mm
- net /G3: track 35.9 -> 28.4 mm
- net /RST: track 27.6 -> 20.1 mm, vias 2 -> 1
- net GND: track 19.2 -> 16.3 mm, vias 8 -> 9
- net /G4: track 45.3 -> 42.5 mm
- net /Rx: track 26.3 -> 28.8 mm, vias 0 -> 1
- net +3.3V: track 12.5 -> 10.2 mm, vias 7 -> 6
- net Net-(D1-Pad2): track 1.77 -> 0.00 mm
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Other:
- net class mainPower: clearance 0.5 -> 1
- board text added: "GPIO0"
- board text added: "RST"
