File: hardware/KiCAD/meross.sch (KiCad schematic (older format))
At the start: 43 parts, among them J1 Conn_01x01_Female, J2 Conn_01x01_Female, J3 Conn_01x04_Male, J4 Conn_01x01_Female, J5 Conn_01x01_Female, J6 Conn_01x01_Female, J7 Conn_01x01_Female, K1 G5Q-1A, K2 G5Q-1A, K3 G5Q-1A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

Commit message: v1.0.0
Parts:
- removed C7: 220uf, Capacitor_THT:CP_Radial_D6.3mm_P2.50mm, symbol Device:CP
- removed D1: D_0001, DVB_LED:LED_0603-red, symbol DVB_D:D_0001
- removed L1: L_0004, DVB_Inductors:L_2020-Vishay, symbol DVB_L:L_0004
- removed R6: R_0027, DVB_Resistors:R_0603, symbol DVB_R:R_0027
- J3: footprint Connector_PinHeader_2.54mm:PinHeader_1x04_P2.54mm_Vertical -> Connector_PinHeader_2.54mm:PinHeader_2x02_P2.54mm_Vertical
- PS1: symbol meross:VTX-214-005-012 -> meross-rescue:VTX-214-005-012-meross
Connections:
- net +12V: now also PS1.5 (DC+V)
- net +3.3V: now also J3.2 (Pin_2); no longer J3.4 (Pin_4)
- net GND: now also SW1.4, SW2.4
- net GPIO0: now also R4.2, SW2.1
- net RST: now also SW1.1
- net Rx: now also J3.4 (Pin_4); no longer J3.2 (Pin_2), R5.2
- net Tx: no longer R4.2
- net at U1.17 (GPIO2): now also R5.2
- no-connect marks 12 -> 9
Other:
- moved on the sheet: R4, R5
Changed lines of the file:
@@
 F 0 "J3" H 4048 6280 50  0000 R CNN
 F 1 "Conn_01x04_Male" H 4048 6371 50  0000 R CNN
-F 2 "Connector_PinHeader_2.54mm:PinHeader_1x04_P2.54mm_Vertical" H 4075 6400 50  0001 C CNN
+F 2 "Connector_PinHeader_2.54mm:PinHeader_2x02_P2.54mm_Vertical" H 4075 6400 50  0001 C CNN
 F 3 "~" H 4075 6400 50  0001 C CNN
 	1    4075 6400
@@
 L DVB_Power:+3.3V #PWR018
 U 1 1 5D5A96C5
-P 3875 6200
-F 0 "#PWR018" H 3875 6130 30  0001 C CNN
-F 1 "+3.3V" H 3875 6338 30  0000 C CNN
-F 2 "" H 3775 6000 50  0001 C CNN
-F 3 "" H 3875 6100 50  0001 C CNN
-	1    3875 6200
+P 3700 6400
+F 0 "#PWR018" H 3700 6330 30  0001 C CNN
+F 1 "+3.3V" H 3700 6538 30  0000 C CNN
+F 2 "" H 3600 6200 50  0001 C CNN
+F 3 "" H 3700 6300 50  0001 C CNN
+	1    3700 6400
 	1    0    0    -1
 $EndComp
 Text Label 3875 6300 2    39   ~ 0
 Tx
-Text Label 3875 6400 2    39   ~ 0
+Text Label 3875 6200 2    39   ~ 0
 Rx
 $Comp
@@
 $EndComp
 $Comp
-L DVB_R:R_0065 R4
-U 1 1 5D5D3A74
-P 4525 3675
-F 0 "R4" H 4600 3675 50  0000 L CNN
-F 1 "R_0065" H 4525 3475 50  0001 C CNN
-F 2 "DVB_Resistors:R_0603" H 4525 3325 50  0001 C CNN
-F 3 "generic" H 4525 3400 50  0001 C CNN
-F 4 "10k" V 4525 3600 50  0000 L CNN "Field4"
-F 5 "5%" V 4275 3575 50  0001 L CNN "Field5"
-F 6 "100mW" V 4350 3575 50  0001 L CNN "Field6"
-	1    4525 3675
-	1    0    0    -1
-$EndComp
-$Comp
-L DVB_R:R_0065 R5
-U 1 1 5D5D3B44
-P 4775 3675
-F 0 "R5" H 4850 3675 50  0000 L CNN
-F 1 "R_0065" H 4775 3475 50  0001 C CNN
-F 2 "DVB_Resistors:R_0603" H 4775 3325 50  0001 C CNN
-F 3 "generic" H 4775 3400 50  0001 C CNN
-F 4 "10k" V 4775 3600 50  0000 L CNN "Field4"
-F 5 "5%" V 4525 3575 50  0001 L CNN "Field5"
-F 6 "100mW" V 4600 3575 50  0001 L CNN "Field6"
-	1    4775 3675
-	1    0    0    -1
-$EndComp
-Wire Wire Line
-	4175 4025 4775 4025
-Wire Wire Line
-	4775 4025 4775 3825
-$Comp
 L DVB_C:C_0037 C2
 U 1 1 5D5E8FA6
@@
 L DVB_Power:+3.3V #PWR013
 U 1 1 5D5ED68C
-P 4525 3525
-F 0 "#PWR013" H 4525 3455 30  0001 C CNN
-F 1 "+3.3V" H 4525 3663 30  0000 C CNN
-F 2 "" H 4425 3325 50  0001 C CNN
-F 3 "" H 4525 3425 50  0001 C CNN
-	1    4525 3525
+P 4525 3275
+F 0 "#PWR013" H 4525 3205 30  0001 C CNN
+F 1 "+3.3V" H 4525 3413 30  0000 C CNN
+F 2 "" H 4425 3075 50  0001 C CNN
+F 3 "" H 4525 3175 50  0001 C CNN
+	1    4525 3275
 	1    0    0    -1
 $EndComp
 Text Label 4175 3725 0    39   ~ 0
 GPIO0
-Wire Wire Line
-	4175 3825 4525 3825
-Wire Wire Line
-	4525 3525 4775 3525
-Connection ~ 4525 3525
 $Comp
 L DVB_Power:GND #PWR01
@@
 Text Label 1350 6125 2    39   ~ 0
 RST
-NoConn ~ 1750 6125
-NoConn ~ 1750 6525
 $Comp
 L DVB_C:C_0029 C1
@@
 Text Label 2675 6125 2    39   ~ 0
 GPIO0
-NoConn ~ 3075 6125
-NoConn ~ 3075 6525
 $Comp
 L DVB_C:C_0029 C3
@@
 Wire Wire Line
 	2675 6525 2875 6525
-Connection ~ 2875 6525
-$Comp
-L DVB_D:D_0001 D1
-U 1 1 5D5FFE1D
-P 4550 4225
-F 0 "D1" H 4550 4325 50  0000 C CNN
-F 1 "D_0001" H 4550 4075 50  0001 C CNN
-F 2 "DVB_LED:LED_0603-red" H 4550 3975 50  0001 C CNN
-F 3 "http://www.vishay.com/docs/83172/tlmo1000.pdf" H 4550 3875 50  0001 C CNN
-F 4 "TLMS1000-GS08" H 4550 3775 50  0001 C CNN "Field4"
-F 5 "2mA" H 4550 3575 50  0001 C CNN "Field5"
-F 6 "LED" H 4550 3675 50  0001 C CNN "Field6"
-F 7 "RED" H 4550 4100 50  0000 C CNN "Field7"
-F 8 "TOP" H 4550 3475 50  0001 C CNN "Field8"
-	1    4550 4225
-	1    0    0    -1
-$EndComp
-$Comp
-L DVB_R:R_0027 R6
-U 1 1 5D60093C
-P 4850 4225
-F 0 "R6" V 4750 4225 50  0000 C CNN
-F 1 "R_0027" H 4850 4025 50  0001 C CNN
-F 2 "DVB_Resistors:R_0603" H 4850 3875 50  0001 C CNN
-F 3 "generic" H 4850 3950 50  0001 C CNN
-F 4 "220" V 4850 4225 50  0000 C CNN "Field4"
-F 5 "1%" V 4600 4125 50  0001 L CNN "Field5"
-F 6 "100mW" V 4675 4125 50  0001 L CNN "Field6"
-	1    4850 4225
-	0    1    1    0
-$EndComp
-$Comp
-L DVB_Power:+3.3V #PWR017
-U 1 1 5D601797
-P 5000 4225
-F 0 "#PWR017" H 5000 4155 30  0001 C CNN
-F 1 "+3.3V" H 5000 4363 30  0000 C CNN
-F 2 "" H 4900 4025 50  0001 C CNN
-F 3 "" H 5000 4125 50  0001 C CNN
-	1    5000 4225
-	1    0    0    -1
-$EndComp
-$Comp
-L meross:VTX-214-005-012 PS1
+$Comp
+L meross-rescue:VTX-214-005-012-meross PS1
 U 1 1 5D6062E8
 P 2025 1200
@@
 Wire Wire Line
 	4175 4625 4350 4625
-Wire Wire Line
-	4400 4225 4175 4225
 NoConn ~ 4175 4125
 NoConn ~ 2975 4325
@@
 NoConn ~ 2975 4725
 NoConn ~ 2975 4825
-$Comp
-L DVB_L:L_0004 L1
-U 1 1 5D60CB8E
-P 2575 1100
-F 0 "L1" H 2575 1380 50  0000 C CNN
-F 1 "L_0004" H 2575 900 50  0001 C CNN
-F 2 "DVB_Inductors:L_2020-Vishay" H 2575 825 50  0001 C CNN
-F 3 "http://www.farnell.com/datasheets/2050374.pdf?_ga=2.106835719.526238941.1497949497-421346633.1483631847" H 2575 750 50  0001 C CNN
-F 4 "IHLP2020BZER4R7M01" H 2575 675 50  0001 C CNN "Field4"
-F 5 "5A" H 2575 1289 50  0000 C CNN "Field5"
-F 6 "COIL" H 2575 600 50  0001 C CNN "Field6"
-F 7 "4.7µH" H 2575 1198 50  0000 C CNN "Field7"
-	1    2575 1100
-	1    0    0    -1
-$EndComp
-$Comp
-L Device:CP C7
-U 1 1 5D60D031
-P 2725 1250
-F 0 "C7" H 2843 1296 50  0000 L CNN
-F 1 "220uf" H 2843 1205 50  0000 L CNN
-F 2 "Capacitor_THT:CP_Radial_D6.3mm_P2.50mm" H 2763 1100 50  0001 C CNN
-F 3 "~" H 2725 1250 50  0001 C CNN
-	1    2725 1250
-	1    0    0    -1
-$EndComp
-Connection ~ 2725 1100
-$Comp
-L DVB_Power:GND #PWR0101
-U 1 1 5D60D425
-P 2725 1400
-F 0 "#PWR0101" H 2725 1240 30  0001 C CNN
-F 1 "GND" H 2729 1262 30  0000 C CNN
-F 2 "" H 2625 1050 50  0001 C CNN
-F 3 "" H 2725 1150 50  0001 C CNN
-	1    2725 1400
-	1    0    0    -1
-$EndComp
 Connection ~ 3425 1100
 Connection ~ 3025 1100
 Wire Wire Line
 	3025 1100 3425 1100
-Wire Wire Line
-	2725 1100 3025 1100
 Wire Notes Line
 	875  5950 3575 5950
@@
 	-1   0    0    1
 $EndComp
+Wire Wire Line
+	3700 6400 3875 6400
+Wire Wire Line
+	2425 1100 3025 1100
+Connection ~ 2875 6525
+Wire Wire Line
+	2875 6125 3075 6125
+Connection ~ 2875 6125
+Wire Wire Line
+	3075 6525 2875 6525
+Wire Wire Line
+	1750 6125 1550 6125
+Connection ~ 1550 6125
+Wire Wire Line
+	1550 6525 1750 6525
+NoConn ~ 4175 4225
+$Comp
+L DVB_R:R_0065 R5
+U 1 1 5D5D3B44
+P 4775 3425
+F 0 "R5" V 4675 3375 50  0000 L CNN
+F 1 "R_0065" H 4775 3225 50  0001 C CNN
+F 2 "DVB_Resistors:R_0603" H 4775 3075 50  0001 C CNN
+F 3 "generic" H 4775 3150 50  0001 C CNN
+F 4 "10k" V 4775 3350 50  0000 L CNN "Field4"
+F 5 "5%" V 4525 3325 50  0001 L CNN "Field5"
+F 6 "100mW" V 4600 3325 50  0001 L CNN "Field6"
+	1    4775 3425
+	1    0    0    -1
+$EndComp
+Wire Wire Line
+	4525 3275 4775 3275
+Connection ~ 4525 3275
+$Comp
+L DVB_R:R_0065 R4
+U 1 1 5D5D3A74
+P 4525 3425
+F 0 "R4" V 4425 3375 50  0000 L CNN
+F 1 "R_0065" H 4525 3225 50  0001 C CNN
+F 2 "DVB_Resistors:R_0603" H 4525 3075 50  0001 C CNN
+F 3 "generic" H 4525 3150 50  0001 C CNN
+F 4 "10k" V 4525 3350 50  0000 L CNN "Field4"
+F 5 "5%" V 4275 3325 50  0001 L CNN "Field5"
+F 6 "100mW" V 4350 3325 50  0001 L CNN "Field6"
+	1    4525 3425
+	1    0    0    -1
+$EndComp
+Wire Wire Line
+	4175 3725 4525 3725
+Wire Wire Line
+	4525 3725 4525 3575
+Wire Wire Line
+	4775 3575 4775 3925
+Wire Wire Line
+	4775 3925 4175 3925
 $EndSCHEMATC
